Commit message: Added robotiq gripper to xacro model

File: cob_hardware_config/raw3-6/urdf/raw3-6.urdf.xacro (robot description, xacro)
@@ -12,4 +12,6 @@
   <!-- ur10 -->
   <xacro:include filename="$(find cob_description)/urdf/ur_arm/ur10_arm.urdf.xacro" />
+  <!-- robotiq gripper -->
+  <xacro:include filename="$(find robotiq_s_model_visualization)/cfg/robotiq_hand_macro.urdf.xacro" />
   <!-- composition of the robot -->
   <xacro:raw_base name="base"/>
@@ -26,4 +28,7 @@
     <origin xyz="${arm_x} ${arm_y} ${arm_z}" rpy="${arm_roll} ${arm_pitch} ${arm_yaw}" />
   </xacro:ur10>
+  <xacro:robotiq_hand prefix="gripper_" parent="arm_tool0" reflect="0">
+    <origin xyz="0 0 .05" rpy="1.570795 0 -1.570795"/>
+  </xacro:robotiq_hand>
   <gazebo>
     <plugin name="ros_control" filename="libhwi_switch_gazebo_ros_control.so">
