Commit message: init from brad's code in cob

File: cob_hardware_config/raw3-6/urdf/no_realsense-raw3-6-urdf.xacro (robot description, xacro)
@@ -14,6 +14,4 @@
   <!-- robotiq gripper -->
   <xacro:include filename="$(find robotiq_s_model_visualization)/cfg/robotiq_hand_macro.urdf.xacro" />
-  <!-- RealSense Sensors -->
-  <xacro:include filename="$(find yuri)/urdf/realsense/r200.urdf.xacro"/>
   <!-- composition of the robot -->
   <xacro:raw_base name="base"/>
@@ -34,9 +32,4 @@
     <!--<origin xyz="0 0 .05" rpy="1.570795 0 -1.570795"/>-->
   </xacro:robotiq_hand>
-<!--
-  <xacro:sensor_r200 prefix="vision_wrist_" parent="arm_tool0">
-    <origin xyz="0 -0.3 .15" rpy="1.570795 0 -0.7753975"/>
-  </xacro:sensor_r200>
--->
   <gazebo>
     <plugin name="ros_control" filename="libhwi_switch_gazebo_ros_control.so">
