Commit message: add sick sensor in robot base urdf, move sr200 to cob_common

File: cob_hardware_config/robots/raw3-6/urdf/properties.urdf.xacro (robot description, xacro)
@@ -7,4 +7,5 @@
 	<!-- ***************** -->
 	<!-- laser front mount positions | relative to base_link -->
+    <!--XXX: these parameters e.g. def_laser_front_x are from cob_robots/cob_hardware_config/robots/raw3-5/urdf/calibration_default.urdf.xacro-->
 	<property name="laser_front_x" value="${def_laser_front_x+offset_laser_front_x}"/>
 	<property name="laser_front_y" value="${def_laser_front_y+offset_laser_front_y}"/>

File: cob_hardware_config/robots/raw3-6/urdf/raw3-6.urdf.xacro (robot description, xacro)
@@ -10,9 +10,11 @@
   <xacro:include filename="$(find raw_description)/urdf/tower_symetric/tower.urdf.xacro" />
   <!-- ur10 -->
-  <xacro:include filename="$(find cob_description)/urdf/ur_arm/ur10_arm.urdf.xacro" />
+  <xacro:include filename="$(find raw_description)/urdf/ur_arm/ur10_arm.urdf.xacro" />
   <!-- robotiq gripper -->
   <xacro:include filename="$(find robotiq_s_model_visualization)/cfg/robotiq_hand_macro.urdf.xacro" />
   <!-- RealSense Sensors -->
-  <xacro:include filename="$(find cob_hardware_config)/robots/raw3-6/realsense/r200.urdf.xacro"/>
+  <xacro:include filename="$(find cob_description)/urdf/sensors/r200.urdf.xacro"/>
+  <!-- sick s300 -->
+  <xacro:include filename="$(find cob_description)/urdf/sensors/sick_s300_laser.urdf.xacro"/>
   <!-- composition of the robot -->
   <xacro:raw_base name="base"/>
@@ -33,9 +35,17 @@
     <!--<origin xyz="0 0 .05" rpy="1.570795 0 -1.570795"/>-->
   </xacro:robotiq_hand>
-<!--
+  <!-- sick s300 -->
+  <!--XXX: these parameters are from cob_robots/cob_hardware_config/robots/raw3-5/urdf/properties.urdf.xacro-->
+  <xacro:sick_s300_laser_v0 name="base_laser_front" parent="base">
+    <origin xyz="${laser_front_x} ${laser_front_y} ${laser_front_z}" rpy="${laser_front_roll} ${laser_front_pitch} ${laser_front_yaw}" />
+  </xacro:sick_s300_laser_v0>
+  <xacro:sick_s300_laser_v0 name="base_laser_rear" parent="base">
+    <origin xyz="${laser_rear_x} ${laser_rear_y} ${laser_rear_z}" rpy="${laser_rear_roll} ${laser_rear_pitch} ${laser_rear_yaw}" />
+  </xacro:sick_s300_laser_v0>
+  <!--
   <xacro:sensor_r200 prefix="vision_wrist_" parent="arm_tool0">
     <origin xyz="0 -0.3 .15" rpy="1.570795 0 -0.7753975"/>
   </xacro:sensor_r200>
--->
+  -->
   <gazebo>
     <plugin name="ros_control" filename="libhwi_switch_gazebo_ros_control.so">
