Commit message: add jennifer gazebo plugin for grasp, not work well in gazebo2

File: cob_hardware_config/robots/raw3-6/urdf/raw3-6.urdf.xacro (robot description, xacro)
@@ -1,162 +1,224 @@
 <?xml version="1.0"?>
 <robot xmlns:xacro="http://www.ros.org/wiki/xacro"
-             name="raw3-6" >
-    <arg name="load_wrist_sr300_simulator" default="$(optenv LOAD_WRIST_SR300_SIMULATOR !!NO_LOAD_WRIST_SR300_SIMULATOR_SET!!)"/>
-    <arg name="visualize_wrist_sr300_simulator" default="$(optenv VISUALIZE_WRIST_SR300_SIMULATOR !!NO_VISUALIZE_WRIST_SR300_SIMULATOR_SET!!)"/>
-    <arg name="visualize_sick_s300_simulator" default="$(optenv VISUALIZE_SICK_S300_SIMULATOR !!NO_VISUALIZE_SICK_S300_SIMULATOR_SET!!)"/>
-    <arg name="sim" default="$(optenv SIM !!NO_SIM_SET!!)"/>
-    <!-- common stuff -->
-    <xacro:include filename="$(find cob_description)/urdf/common.xacro" />
-    <xacro:include filename="$(find cob_description)/urdf/materials.urdf.xacro" />
-    <xacro:include filename="$(find cob_hardware_config)/robots/raw3-6/urdf/properties.urdf.xacro" />
-    <!-- raw base -->
-    <xacro:include filename="$(find raw_description)/urdf/base_long/base.urdf.xacro" />
-    <!-- raw tower -->
-    <xacro:include filename="$(find raw_description)/urdf/tower_symetric/tower.urdf.xacro" />
-    <!-- ur10 -->
-    <xacro:include filename="$(find cob_description)/urdf/ur_arm/ur10_arm.urdf.xacro" />
-    <!-- robotiq gripper -->
-    <xacro:include filename="$(find cob_description)/urdf/robotiq_gripper/robotiq_s_gripper.urdf.xacro" />
-    <!-- RealSense Sensors -->
-    <!--<xacro:include filename="$(find cob_description)/urdf/sensors/r200.urdf.xacro"/>-->
-    <xacro:include filename="$(find cob_description)/urdf/sensors/realsense.urdf.xacro"/>
-    <xacro:include filename="$(find cob_description)/urdf/sensors/realsense.gazebo.xacro"/>
-    <!-- sick s300 -->
-    <xacro:include filename="$(find cob_description)/urdf/sensors/sick_s300_laser.urdf.xacro"/>
-    <!-- composition of the robot -->
-    <xacro:raw_base sim="$(arg sim)" visualize_sick_s300_simulator="$(arg visualize_sick_s300_simulator)" name="base"/>
-    <!-- These are already defined at ./src/cob_common/raw_description/urdf/base_long/base.urdf.xacro. -->
-    <!-- These are already defined at ./src/cob_common/raw_description/urdf/base_short/base.urdf.xacro. -->
-    <!-- base laser front -->
-    <!--XXX: these parameters are from cob_robots/cob_hardware_config/robots/raw3-5/urdf/properties.urdf.xacro-->
-    <!-- <xacro:sick_s300_laser_v0 name="base_laser_front" parent="base">
-        <origin xyz="${laser_front_x} ${laser_front_y} ${laser_front_z}" rpy="${laser_front_roll} ${laser_front_pitch} ${laser_front_yaw}" />
-    </xacro:sick_s300_laser_v0> -->
-    <!-- base laser rear -->
-    <!-- <xacro:sick_s300_laser_v0 name="base_laser_rear" parent="base">
-        <origin xyz="${laser_rear_x} ${laser_rear_y} ${laser_rear_z}" rpy="${laser_rear_roll} ${laser_rear_pitch} ${laser_rear_yaw}" />
-    </xacro:sick_s300_laser_v0> -->
-    <xacro:tower_symetric name="tower" parent="base_link">
-            <origin xyz="${tower_x} ${tower_y} ${tower_z}" rpy="${tower_roll} ${tower_pitch} ${tower_yaw}" />
-    </xacro:tower_symetric>
-    <xacro:ur10 name="arm" parent="base_link" sim="$(arg sim)">
-        <origin xyz="${arm_x} ${arm_y} ${arm_z}" rpy="${arm_roll} ${arm_pitch} ${arm_yaw}" />
-    </xacro:ur10>
-    <!--directlt defined here instead of retrieving from-->
-    <!--$(find cob_hardware_config)/robots/raw3-6/urdf/properties.urdf.xacro-->
-    <!--it has to be arm_tool0 instead of arm_ee_link-->
-    <!--<xacro:robotiq_hand prefix="gripper_" parent="arm_wrist_extension" reflect="0">-->
-        <!--<origin xyz="0 0 .05" rpy="1.570795 0 -0.7753975"/>-->
-    <!--</xacro:robotiq_hand>-->
-    <xacro:robotiq name="gripper" parent="arm_tool0" reflect="0" sim="$(arg sim)">
-    <!--<xacro:robotiq_hand prefix="gripper_" parent="arm_tool0" reflect="0">-->
-        <!-- We have to rotate the gripper by 45 around z, so that it matches the real robot -->
-        <origin xyz="0 0 .05" rpy="${90/180*pi} 0 -${45/180*pi}"/>
-        <!--<origin xyz="0 0 .05" rpy="${90/180*pi} 0 -1.570795"/>-->
-    </xacro:robotiq>
-    <!-- >>>>>>>>>>>>>>>>>>>>>>>>>>>>>>>>>>>>>>>>>>>>>>>>>>>>>>>>>>>>>>>>>> -->
-    <!-- wrist_sr300 mount and camera -->
-    <!--we add the sensor above the robot base metal board-->
-    <!--x = in the middle of the base metal board-->
-    <!--z = as high as the arm shoulder square base-->
-    <!--y = in the middle of the 2 batteries under the base metal board-->
-    <!--z - blue axis - larger is going up-->
-    <!--x - red axis - larger is going forward the robot-->
-    <!--y - green axis - larger is going left to robot-->
-    <!--yaw - rotate around z, 1.57 is 90 degree, so the camera is facing to the right-->
-    <joint name="wrist_sr300_realsense_mount_joint" type="fixed">
-        <!--<xacro:insert_block name="origin" />-->
-        <parent link="arm_tool0"/>
-        <child link="wrist_sr300_realsense_mount_link"/>
-        <!--always in parent reference frame-->
-        <!-- we have to rotate 45 around z to match the robotiq, while the robotiq has to rotate the same to match the real robot -->
-        <origin xyz="0.05 0.065 0.0025" rpy="0 0 -${45/180*pi}" />
-        <!-- <origin xyz="0.0 0.075 0.0025" rpy="0 0 0" /> -->
-        <!--for prismatic and revolute (in local joint reference frame)-->
-        <!--<axis xyz="0 0 1" />-->
-    </joint>
-    <link name="wrist_sr300_realsense_mount_link" >
-        <inertial>
-            <mass value="0.1"/>
-            <origin xyz="0 0 0"/>
-            <!--https://gist.github.com/awesomebytes/39a4ba6c64956a1aa9bd-->
-            <inertia ixx="0.00018" ixy="0.0" ixz="0.0" iyy="0.00002" iyz="0.0" izz="0.0002" />
-        </inertial>
-        <visual>
-            <origin xyz="0.0 0.0 0.0" rpy="0 0 0"/>
-            <geometry>
-                <box size="0.05 0.150 0.005"/>
-            </geometry>
-            <material name="gray">
-                <color rgba="0.50 0.50 0.50 1" />
-                <!-- <color rgba="1.0 1.0 1.0 1" /> -->
-                <!--<color rgba="0.2 0.2 1 1" />-->
-            </material>
-        </visual>
-        <collision>
-            <origin xyz="0.0 0.0 0.0" rpy="0 0 0"/>
-            <geometry>
-                <box size="0.05 0.150 0.005"/>
-            </geometry>
-        </collision>
-    </link>
-    <!-- the view of the camera is only determined by the following xyzrpy -->
-    <!-- it is not determined by the xyzrpy in realsense.gazebo,xacro and realsense.urdf.xacro -->
-    <!-- because everything inside realsense.gazebo,xacro and realsense.urdf.xacro are used for visualizing the camera. What the camera will see will not be influenced by its visualization parameters. -->
-    <xacro:property name="wrist_sr300_name" value="wrist_sr300_realsense" />
-    <!-- The rpy for simulation is different from the rpy setup for the actual camera. If we use the rpy from actual camera in simulation, the view will be wrong -->
-    <!-- gazebo plug-in for simulating the camera -->
-    <xacro:if value="$(arg load_wrist_sr300_simulator)">
-      <xacro:realsense
-        sim="$(arg load_wrist_sr300_simulator)"
-        name="${wrist_sr300_name}"
-        parent="wrist_sr300_realsense_mount_link">
-          <!-- <origin xyz="0.0 0.065 0.038" rpy="0.0 -${90/180*pi} -${90/180*pi}"/> -->
-          <origin xyz="0.0 0.065 0.038" rpy="0.0 0.0 ${180/180*pi}"/>
-      </xacro:realsense>
-      <xacro:realsense_rgb_gazebo_v0
-        name="${wrist_sr300_name}"
-        link_name="${wrist_sr300_name}_rgb_frame"
-        frame_name="${wrist_sr300_name}_rgb_optical_frame"
-        camera_name="${wrist_sr300_name}"
-        visualize_wrist_sr300_simulator="$(arg visualize_wrist_sr300_simulator)" />
-      <xacro:realsense_ir_gazebo_v0
-        name="${wrist_sr300_name}"
-        link_name="${wrist_sr300_name}_depth_frame"
-        frame_name="${wrist_sr300_name}_depth_optical_frame"
-        camera_name="${wrist_sr300_name}"
-        visualize_wrist_sr300_simulator="$(arg visualize_wrist_sr300_simulator)" />
-    </xacro:if>
-    <!-- if not in simulation: -->
-    <xacro:unless value="$(arg load_wrist_sr300_simulator)">
-      <xacro:realsense
-        sim="$(arg load_wrist_sr300_simulator)"
-        name="${wrist_sr300_name}"
-        parent="wrist_sr300_realsense_mount_link">
-          <!--<origin xyz="0. -0.25 0.5" rpy="0.0 0.0 -1.57"/>-->
-          <origin xyz="0.0 0.065 0.038" rpy="0.0 0.0 ${180/180*pi}"/>
-      </xacro:realsense>
-    </xacro:unless>
-    <!--
-    <xacro:sensor_r200 prefix="vision_wrist_" parent="arm_tool0">
-        <origin xyz="0 -0.3 .15" rpy="1.570795 0 -0.7753975"/>
-    </xacro:sensor_r200>
-    -->
-    <!-- <<<<<<<<<<<<<<<<<<<<<<<<<<<<<<<<<<<<<<<<<<<<<<<<<<<<<<<<<<<<<<<<<< -->
-    <!--
+       name="raw3-6" >
+  <arg name="load_wrist_sr300_simulator" default="$(optenv LOAD_WRIST_SR300_SIMULATOR !!NO_LOAD_WRIST_SR300_SIMULATOR_SET!!)"/>
+  <arg name="visualize_wrist_sr300_simulator" default="$(optenv VISUALIZE_WRIST_SR300_SIMULATOR !!NO_VISUALIZE_WRIST_SR300_SIMULATOR_SET!!)"/>
+  <arg name="visualize_sick_s300_simulator" default="$(optenv VISUALIZE_SICK_S300_SIMULATOR !!NO_VISUALIZE_SICK_S300_SIMULATOR_SET!!)"/>
+  <arg name="sim" default="$(optenv SIM !!NO_SIM_SET!!)"/>
+  <!-- common stuff -->
+  <xacro:include filename="$(find cob_description)/urdf/common.xacro" />
+  <xacro:include filename="$(find cob_description)/urdf/materials.urdf.xacro" />
+  <xacro:include filename="$(find cob_hardware_config)/robots/raw3-6/urdf/properties.urdf.xacro" />
+  <!-- raw base -->
+  <xacro:include filename="$(find raw_description)/urdf/base_long/base.urdf.xacro" />
+  <!-- raw tower -->
+  <xacro:include filename="$(find raw_description)/urdf/tower_symetric/tower.urdf.xacro" />
+  <!-- ur10 -->
+  <xacro:include filename="$(find cob_description)/urdf/ur_arm/ur10_arm.urdf.xacro" />
+  <!-- robotiq gripper -->
+  <xacro:include filename="$(find cob_description)/urdf/robotiq_gripper/robotiq_s_gripper.urdf.xacro" />
+  <!-- RealSense Sensors -->
+  <!--<xacro:include filename="$(find cob_description)/urdf/sensors/r200.urdf.xacro"/>-->
+  <xacro:include filename="$(find cob_description)/urdf/sensors/realsense.urdf.xacro"/>
+  <xacro:include filename="$(find cob_description)/urdf/sensors/realsense.gazebo.xacro"/>
+  <!-- sick s300 -->
+  <xacro:include filename="$(find cob_description)/urdf/sensors/sick_s300_laser.urdf.xacro"/>
+  <!-- composition of the robot -->
+  <xacro:raw_base sim="$(arg sim)" visualize_sick_s300_simulator="$(arg visualize_sick_s300_simulator)" name="base"/>
+  <!-- These are already defined at ./src/cob_common/raw_description/urdf/base_long/base.urdf.xacro. -->
+  <!-- These are already defined at ./src/cob_common/raw_description/urdf/base_short/base.urdf.xacro. -->
+  <!-- base laser front -->
+  <!--XXX: these parameters are from cob_robots/cob_hardware_config/robots/raw3-5/urdf/properties.urdf.xacro-->
+  <!-- <xacro:sick_s300_laser_v0 name="base_laser_front" parent="base">
+    <origin xyz="${laser_front_x} ${laser_front_y} ${laser_front_z}" rpy="${laser_front_roll} ${laser_front_pitch} ${laser_front_yaw}" />
+  </xacro:sick_s300_laser_v0> -->
+  <!-- base laser rear -->
+  <!-- <xacro:sick_s300_laser_v0 name="base_laser_rear" parent="base">
+    <origin xyz="${laser_rear_x} ${laser_rear_y} ${laser_rear_z}" rpy="${laser_rear_roll} ${laser_rear_pitch} ${laser_rear_yaw}" />
+  </xacro:sick_s300_laser_v0> -->
+  <xacro:tower_symetric name="tower" parent="base_link">
+      <origin xyz="${tower_x} ${tower_y} ${tower_z}" rpy="${tower_roll} ${tower_pitch} ${tower_yaw}" />
+  </xacro:tower_symetric>
+  <xacro:ur10 name="arm" parent="base_link" sim="$(arg sim)">
+    <origin xyz="${arm_x} ${arm_y} ${arm_z}" rpy="${arm_roll} ${arm_pitch} ${arm_yaw}" />
+  </xacro:ur10>
+  <!--directlt defined here instead of retrieving from-->
+  <!--$(find cob_hardware_config)/robots/raw3-6/urdf/properties.urdf.xacro-->
+  <!--it has to be arm_tool0 instead of arm_ee_link-->
+  <!--<xacro:robotiq_hand prefix="gripper_" parent="arm_wrist_extension" reflect="0">-->
+    <!--<origin xyz="0 0 .05" rpy="1.570795 0 -0.7753975"/>-->
+  <!--</xacro:robotiq_hand>-->
+  <xacro:robotiq name="gripper" parent="arm_tool0" reflect="0" sim="$(arg sim)">
+  <!--<xacro:robotiq_hand prefix="gripper_" parent="arm_tool0" reflect="0">-->
+    <!-- We have to rotate the gripper by 45 around z, so that it matches the real robot -->
+    <origin xyz="0 0 .05" rpy="${90/180*pi} 0 -${45/180*pi}"/>
+    <!--<origin xyz="0 0 .05" rpy="${90/180*pi} 0 -1.570795"/>-->
+  </xacro:robotiq>
+  <!-- >>>>>>>>>>>>>>>>>>>>>>>>>>>>>>>>>>>>>>>>>>>>>>>>>>>>>>>>>>>>>>>>>> -->
+  <!-- wrist_sr300 mount and camera -->
+  <!--we add the sensor above the robot base metal board-->
+  <!--x = in the middle of the base metal board-->
+  <!--z = as high as the arm shoulder square base-->
+  <!--y = in the middle of the 2 batteries under the base metal board-->
+  <!--z - blue axis - larger is going up-->
+  <!--x - red axis - larger is going forward the robot-->
+  <!--y - green axis - larger is going left to robot-->
+  <!--yaw - rotate around z, 1.57 is 90 degree, so the camera is facing to the right-->
+  <joint name="wrist_sr300_realsense_mount_joint" type="fixed">
+    <!--<xacro:insert_block name="origin" />-->
+    <parent link="arm_tool0"/>
+    <child link="wrist_sr300_realsense_mount_link"/>
+    <!--always in parent reference frame-->
+    <!-- we have to rotate 45 around z to match the robotiq, while the robotiq has to rotate the same to match the real robot -->
+    <origin xyz="0.05 0.065 0.0025" rpy="0 0 -${45/180*pi}" />
+    <!-- <origin xyz="0.0 0.075 0.0025" rpy="0 0 0" /> -->
+    <!--for prismatic and revolute (in local joint reference frame)-->
+    <!--<axis xyz="0 0 1" />-->
+  </joint>
+  <link name="wrist_sr300_realsense_mount_link" >
+    <inertial>
+      <mass value="0.1"/>
+      <origin xyz="0 0 0"/>
+      <!--https://gist.github.com/awesomebytes/39a4ba6c64956a1aa9bd-->
+      <inertia ixx="0.00018" ixy="0.0" ixz="0.0" iyy="0.00002" iyz="0.0" izz="0.0002" />
+    </inertial>
+    <visual>
+      <origin xyz="0.0 0.0 0.0" rpy="0 0 0"/>
+      <geometry>
+        <box size="0.05 0.150 0.005"/>
+      </geometry>
+      <material name="gray">
+        <color rgba="0.50 0.50 0.50 1" />
+        <!-- <color rgba="1.0 1.0 1.0 1" /> -->
+        <!--<color rgba="0.2 0.2 1 1" />-->
+      </material>
+    </visual>
+    <collision>
+      <origin xyz="0.0 0.0 0.0" rpy="0 0 0"/>
+      <geometry>
+        <box size="0.05 0.150 0.005"/>
+      </geometry>
+    </collision>
+  </link>
+  <!-- the view of the camera is only determined by the following xyzrpy -->
+  <!-- it is not determined by the xyzrpy in realsense.gazebo,xacro and realsense.urdf.xacro -->
+  <!-- because everything inside realsense.gazebo,xacro and realsense.urdf.xacro are used for visualizing the camera. What the camera will see will not be influenced by its visualization parameters. -->
+  <xacro:property name="wrist_sr300_name" value="wrist_sr300_realsense" />
+  <xacro:property name="realsense_xyz" value="0.0 0.065 0.052"/>
+  <xacro:property name="realsense_rpy" value="0.0 0.0 ${180/180*pi}"/>
+  <!-- The rpy for simulation is different from the rpy setup for the actual camera. If we use the rpy from actual camera in simulation, the view will be wrong -->
+  <!-- gazebo plug-in for simulating the camera -->
+  <xacro:if value="$(arg load_wrist_sr300_simulator)">
+    <xacro:realsense
+    sim="$(arg load_wrist_sr300_simulator)"
+    name="${wrist_sr300_name}"
+    parent="wrist_sr300_realsense_mount_link">
+      <!-- <origin xyz="0.0 0.065 0.038" rpy="0.0 -${90/180*pi} -${90/180*pi}"/> -->
+      <origin xyz="${realsense_xyz}" rpy="${realsense_rpy}"/>
+    </xacro:realsense>
+    <xacro:realsense_rgb_gazebo_v0
+    name="${wrist_sr300_name}"
+    link_name="${wrist_sr300_name}_rgb_frame"
+    frame_name="${wrist_sr300_name}_rgb_optical_frame"
+    camera_name="${wrist_sr300_name}"
+    visualize_wrist_sr300_simulator="$(arg visualize_wrist_sr300_simulator)" />
+    <xacro:realsense_ir_gazebo_v0
+    name="${wrist_sr300_name}"
+    link_name="${wrist_sr300_name}_depth_frame"
+    frame_name="${wrist_sr300_name}_depth_optical_frame"
+    camera_name="${wrist_sr300_name}"
+    visualize_wrist_sr300_simulator="$(arg visualize_wrist_sr300_simulator)" />
+  </xacro:if>
+  <!-- if not in simulation: -->
+  <xacro:unless value="$(arg load_wrist_sr300_simulator)">
+    <xacro:realsense
+    sim="$(arg load_wrist_sr300_simulator)"
+    name="${wrist_sr300_name}"
+    parent="wrist_sr300_realsense_mount_link">
+      <!--<origin xyz="0. -0.25 0.5" rpy="0.0 0.0 -1.57"/>-->
+      <origin xyz="${realsense_xyz}" rpy="${realsense_rpy}"/>
+    </xacro:realsense>
+  </xacro:unless>
+  <!--
+  <xacro:sensor_r200 prefix="vision_wrist_" parent="arm_tool0">
+    <origin xyz="0 -0.3 .15" rpy="1.570795 0 -0.7753975"/>
+  </xacro:sensor_r200>
+  -->
+  <!-- <<<<<<<<<<<<<<<<<<<<<<<<<<<<<<<<<<<<<<<<<<<<<<<<<<<<<<<<<<<<<<<<<< -->
+  <!--
+  <gazebo>
+    <plugin name="ros_control" filename="libhwi_switch_gazebo_ros_control.so">
+      <robotNamespace>base</robotNamespace>
+      <filterJointsParam>joint_names</filterJointsParam>
+    </plugin>
+  </gazebo>
+  -->
+  <!--
+  <gazebo>
+    <plugin name="ros_control" filename="libhwi_switch_gazebo_ros_control.so">
+      <robotNamespace>arm</robotNamespace>
+      <filterJointsParam>joint_names</filterJointsParam>
+    </plugin>
+  </gazebo>
+  -->
+  <!-- https://github.com/JenniferBuehler/gazebo-pkgs/wiki/The-Gazebo-grasp-fix-plugin -->
+  <!-- Clone this in your workspace and that's it! -->
+  <!-- https://github.com/JenniferBuehler/gazebo-pkgs -->
+  <!-- TODO: It seems not working well in gazebo 2.0 -->
+  <!-- <xacro:if value="$(arg sim)">
     <gazebo>
-        <plugin name="ros_control" filename="libhwi_switch_gazebo_ros_control.so">
-            <robotNamespace>base</robotNamespace>
-            <filterJointsParam>joint_names</filterJointsParam>
-        </plugin>
+      <plugin name="gazebo_grasp_fix" filename="libgazebo_grasp_fix.so">
+        <arm>
+          <arm_name>UR10_arm1</arm_name>
+            <palm_link>arm_wrist_3_link</palm_link>
+            <gripper_link>gripper_finger_1_link_0</gripper_link>
+            <gripper_link>gripper_finger_1_link_1</gripper_link>
+            <gripper_link>gripper_finger_1_link_2</gripper_link>
+            <gripper_link>gripper_finger_1_link_3</gripper_link>
+            <gripper_link>gripper_finger_1_link_paradistal_hinge</gripper_link>
+            <gripper_link>gripper_finger_1_link_median_actuating_hinge</gripper_link>
+            <gripper_link>gripper_finger_1_link_median_bar</gripper_link>
+            <gripper_link>gripper_finger_1_link_paramedian_hinge</gripper_link>
+            <gripper_link>gripper_finger_1_link_median_bar_underactuated</gripper_link>
+            <gripper_link>gripper_finger_1_link_paraproximal_actuating_hinge</gripper_link>
+            <gripper_link>gripper_finger_1_link_paraproximal_bar</gripper_link>
+            <gripper_link>gripper_finger_1_link_proximal_actuating_hinge</gripper_link>
+            <gripper_link>gripper_finger_1_link_proximal_actuating_bar</gripper_link>
+            <gripper_link>gripper_finger_2_link_0</gripper_link>
+            <gripper_link>gripper_finger_2_link_1</gripper_link>
+            <gripper_link>gripper_finger_2_link_2</gripper_link>
+            <gripper_link>gripper_finger_2_link_3</gripper_link>
+            <gripper_link>gripper_finger_2_link_paradistal_hinge</gripper_link>
+            <gripper_link>gripper_finger_2_link_median_actuating_hinge</gripper_link>
+            <gripper_link>gripper_finger_2_link_median_bar</gripper_link>
+            <gripper_link>gripper_finger_2_link_paramedian_hinge</gripper_link>
+            <gripper_link>gripper_finger_2_link_median_bar_underactuated</gripper_link>
+            <gripper_link>gripper_finger_2_link_paraproximal_actuating_hinge</gripper_link>
+            <gripper_link>gripper_finger_2_link_paraproximal_bar</gripper_link>
+            <gripper_link>gripper_finger_2_link_proximal_actuating_hinge</gripper_link>
+            <gripper_link>gripper_finger_2_link_proximal_actuating_bar</gripper_link>
+            <gripper_link>gripper_finger_middle_link_0</gripper_link>
+            <gripper_link>gripper_finger_middle_link_1</gripper_link>
+            <gripper_link>gripper_finger_middle_link_2</gripper_link>
+            <gripper_link>gripper_finger_middle_link_3</gripper_link>
+            <gripper_link>gripper_finger_middle_link_paradistal_hinge</gripper_link>
+            <gripper_link>gripper_finger_middle_link_median_actuating_hinge</gripper_link>
+            <gripper_link>gripper_finger_middle_link_median_bar</gripper_link>
+            <gripper_link>gripper_finger_middle_link_paramedian_hinge</gripper_link>
+            <gripper_link>gripper_finger_middle_link_median_bar_underactuated</gripper_link>
+            <gripper_link>gripper_finger_middle_link_paraproximal_actuating_hinge</gripper_link>
+            <gripper_link>gripper_finger_middle_link_paraproximal_bar</gripper_link>
+            <gripper_link>gripper_finger_middle_link_proximal_actuating_hinge</gripper_link>
+            <gripper_link>gripper_finger_middle_link_proximal_actuating_bar</gripper_link>
+        </arm>
+        <forces_angle_tolerance>90</forces_angle_tolerance>
+        <update_rate>4</update_rate>
+        <grip_count_threshold>4</grip_count_threshold>
+        <max_grip_count>8</max_grip_count>
+        <release_tolerance>0.10</release_tolerance>
+        <disable_collisions_on_attach>false</disable_collisions_on_attach>
+        <contact_topic>__default_topic__</contact_topic>
+      </plugin>
     </gazebo>
-    -->
-    <!--
-    <gazebo>
-        <plugin name="ros_control" filename="libhwi_switch_gazebo_ros_control.so">
-            <robotNamespace>arm</robotNamespace>
-            <filterJointsParam>joint_names</filterJointsParam>
-        </plugin>
-    </gazebo>
-    -->
+  </xacro:if> -->
 </robot>
