Commit message: change camera pose

File: cob_hardware_config/robots/raw3-6/urdf/raw3-6.urdf.xacro (robot description, xacro)
@@ -65,11 +65,47 @@
   <!--y - green axis - larger is going left to robot-->
   <!--yaw - rotate around z, 1.57 is 90 degree, so the camera is facing to the right-->
+<!--  <joint name="wrist_sr300_realsense_mount_joint" type="fixed">-->
+    <!--[><xacro:insert_block name="origin" /><]-->
+    <!--<parent link="arm_tool0"/>-->
+    <!--<child link="wrist_sr300_realsense_mount_link"/>-->
+    <!--[>always in parent reference frame<]-->
+    <!--[> we have to rotate 45 around z to match the robotiq, while the robotiq has to rotate the same to match the real robot <]-->
+    <!--<origin xyz="0.05 0.065 0.0025" rpy="0 0 -${45/180*pi}" />-->
+    <!--[> <origin xyz="0.0 0.075 0.0025" rpy="0 0 0" /> <]-->
+    <!--[>for prismatic and revolute (in local joint reference frame)<]-->
+    <!--[><axis xyz="0 0 1" /><]-->
+  <!--</joint>-->
+  <!--<link name="wrist_sr300_realsense_mount_link" >-->
+    <!--<inertial>-->
+      <!--<mass value="0.1"/>-->
+      <!--<origin xyz="0 0 0"/>-->
+      <!--[>https://gist.github.com/awesomebytes/39a4ba6c64956a1aa9bd<]-->
+      <!--<inertia ixx="0.00018" ixy="0.0" ixz="0.0" iyy="0.00002" iyz="0.0" izz="0.0002" />-->
+    <!--</inertial>-->
+    <!--<visual>-->
+      <!--<origin xyz="0.0 0.0 0.0" rpy="0 0 0"/>-->
+      <!--<geometry>-->
+        <!--<box size="0.05 0.150 0.005"/>-->
+      <!--</geometry>-->
+      <!--<material name="gray">-->
+        <!--<color rgba="0.50 0.50 0.50 1" />-->
+        <!--[> <color rgba="1.0 1.0 1.0 1" /> <]-->
+        <!--[><color rgba="0.2 0.2 1 1" /><]-->
+      <!--</material>-->
+    <!--</visual>-->
+    <!--<collision>-->
+      <!--<origin xyz="0.0 0.0 0.0" rpy="0 0 0"/>-->
+      <!--<geometry>-->
+        <!--<box size="0.05 0.150 0.005"/>-->
+      <!--</geometry>-->
+    <!--</collision>-->
+  <!--</link>-->
   <joint name="wrist_sr300_realsense_mount_joint" type="fixed">
     <!--<xacro:insert_block name="origin" />-->
-    <parent link="arm_tool0"/>
+    <parent link="gripper_palm"/>
     <child link="wrist_sr300_realsense_mount_link"/>
     <!--always in parent reference frame-->
     <!-- we have to rotate 45 around z to match the robotiq, while the robotiq has to rotate the same to match the real robot -->
-    <origin xyz="0.05 0.065 0.0025" rpy="0 0 -${45/180*pi}" />
+    <origin xyz="0.00 -0.02 -0.05" rpy="-${90/180*pi} 0 0" />
     <!-- <origin xyz="0.0 0.075 0.0025" rpy="0 0 0" /> -->
     <!--for prismatic and revolute (in local joint reference frame)-->
@@ -86,5 +122,5 @@
       <origin xyz="0.0 0.0 0.0" rpy="0 0 0"/>
       <geometry>
-        <box size="0.05 0.150 0.005"/>
+        <box size="0.05 0.08 0.005"/>
       </geometry>
       <material name="gray">
@@ -97,5 +133,5 @@
       <origin xyz="0.0 0.0 0.0" rpy="0 0 0"/>
       <geometry>
-        <box size="0.05 0.150 0.005"/>
+        <box size="0.05 0.08 0.005"/>
       </geometry>
     </collision>
@@ -105,5 +141,7 @@
   <!-- because everything inside realsense.gazebo,xacro and realsense.urdf.xacro are used for visualizing the camera. What the camera will see will not be influenced by its visualization parameters. -->
   <xacro:property name="wrist_sr300_name" value="wrist_sr300_realsense" />
-  <xacro:property name="realsense_xyz" value="0.0 0.065 0.052"/>
+  <!--<xacro:property name="realsense_xyz" value="0.0 0.065 0.052"/>-->
+  <xacro:property name="realsense_xyz" value="0.0 0.04 0.052"/>
+  <!--<xacro:property name="realsense_rpy" value="0.0 0.0 ${180/180*pi}"/>-->
   <xacro:property name="realsense_rpy" value="0.0 0.0 ${180/180*pi}"/>
   <!-- The rpy for simulation is different from the rpy setup for the actual camera. If we use the rpy from actual camera in simulation, the view will be wrong -->

Commit message: update camera pos

File: cob_hardware_config/robots/raw3-6/urdf/raw3-6.urdf.xacro (robot description, xacro)
@@ -142,5 +142,5 @@
   <xacro:property name="wrist_sr300_name" value="wrist_sr300_realsense" />
   <!--<xacro:property name="realsense_xyz" value="0.0 0.065 0.052"/>-->
-  <xacro:property name="realsense_xyz" value="0.0 0.04 0.052"/>
+  <xacro:property name="realsense_xyz" value="0.0 0.02 0.062"/>
   <!--<xacro:property name="realsense_rpy" value="0.0 0.0 ${180/180*pi}"/>-->
   <xacro:property name="realsense_rpy" value="0.0 0.0 ${180/180*pi}"/>

Commit message: update new caera

File: cob_hardware_config/robots/raw3-6/urdf/raw3-6.urdf.xacro (robot description, xacro)
@@ -142,5 +142,5 @@
   <xacro:property name="wrist_sr300_name" value="wrist_sr300_realsense" />
   <!--<xacro:property name="realsense_xyz" value="0.0 0.065 0.052"/>-->
-  <xacro:property name="realsense_xyz" value="0.0 0.02 0.062"/>
+  <xacro:property name="realsense_xyz" value="0.01 0.06 0.062"/>
   <!--<xacro:property name="realsense_rpy" value="0.0 0.0 ${180/180*pi}"/>-->
   <xacro:property name="realsense_rpy" value="0.0 0.0 ${180/180*pi}"/>

Commit message: new camera

File: cob_hardware_config/robots/raw3-6/urdf/raw3-6.urdf.xacro (robot description, xacro)
@@ -142,5 +142,5 @@
   <xacro:property name="wrist_sr300_name" value="wrist_sr300_realsense" />
   <!--<xacro:property name="realsense_xyz" value="0.0 0.065 0.052"/>-->
-  <xacro:property name="realsense_xyz" value="0.01 0.06 0.062"/>
+  <xacro:property name="realsense_xyz" value="0.01 0.06 0.072"/>
   <!--<xacro:property name="realsense_rpy" value="0.0 0.0 ${180/180*pi}"/>-->
   <xacro:property name="realsense_rpy" value="0.0 0.0 ${180/180*pi}"/>

Commit message: refactor wrist_sr300_realsense -> wrist_camera

File: cob_hardware_config/robots/raw3-6/urdf/raw3-6.urdf.xacro (robot description, xacro)
@@ -2,6 +2,6 @@
 <robot xmlns:xacro="http://www.ros.org/wiki/xacro"
        name="raw3-6" >
-  <arg name="load_wrist_sr300_simulator" default="$(optenv LOAD_WRIST_SR300_SIMULATOR !!NO_LOAD_WRIST_SR300_SIMULATOR_SET!!)"/>
-  <arg name="visualize_wrist_sr300_simulator" default="$(optenv VISUALIZE_WRIST_SR300_SIMULATOR !!NO_VISUALIZE_WRIST_SR300_SIMULATOR_SET!!)"/>
+  <arg name="load_wrist_camera_simulator" default="$(optenv LOAD_WRIST_CAMERA_SIMULATOR !!NO_LOAD_WRIST_CAMERA_SIMULATOR_SET!!)"/>
+  <arg name="visualize_wrist_camera_simulator" default="$(optenv VISUALIZE_WRIST_CAMERA_SIMULATOR !!NO_VISUALIZE_WRIST_CAMERA_SIMULATOR_SET!!)"/>
   <arg name="visualize_sick_s300_simulator" default="$(optenv VISUALIZE_SICK_S300_SIMULATOR !!NO_VISUALIZE_SICK_S300_SIMULATOR_SET!!)"/>
   <arg name="sim" default="$(optenv SIM !!NO_SIM_SET!!)"/>
@@ -56,5 +56,5 @@
   </xacro:robotiq>
   <!-- >>>>>>>>>>>>>>>>>>>>>>>>>>>>>>>>>>>>>>>>>>>>>>>>>>>>>>>>>>>>>>>>>> -->
-  <!-- wrist_sr300 mount and camera -->
+  <!-- wrist_camera mount and camera -->
   <!--we add the sensor above the robot base metal board-->
   <!--x = in the middle of the base metal board-->
@@ -65,8 +65,8 @@
   <!--y - green axis - larger is going left to robot-->
   <!--yaw - rotate around z, 1.57 is 90 degree, so the camera is facing to the right-->
-<!--  <joint name="wrist_sr300_realsense_mount_joint" type="fixed">-->
+<!--  <joint name="wrist_camera_mount_joint" type="fixed">-->
     <!--[><xacro:insert_block name="origin" /><]-->
     <!--<parent link="arm_tool0"/>-->
-    <!--<child link="wrist_sr300_realsense_mount_link"/>-->
+    <!--<child link="wrist_camera_mount_link"/>-->
     <!--[>always in parent reference frame<]-->
     <!--[> we have to rotate 45 around z to match the robotiq, while the robotiq has to rotate the same to match the real robot <]-->
@@ -76,5 +76,5 @@
     <!--[><axis xyz="0 0 1" /><]-->
   <!--</joint>-->
-  <!--<link name="wrist_sr300_realsense_mount_link" >-->
+  <!--<link name="wrist_camera_mount_link" >-->
     <!--<inertial>-->
       <!--<mass value="0.1"/>-->
@@ -101,8 +101,8 @@
     <!--</collision>-->
   <!--</link>-->
-  <joint name="wrist_sr300_realsense_mount_joint" type="fixed">
+  <joint name="wrist_camera_mount_joint" type="fixed">
     <!--<xacro:insert_block name="origin" />-->
     <parent link="gripper_palm"/>
-    <child link="wrist_sr300_realsense_mount_link"/>
+    <child link="wrist_camera_mount_link"/>
     <!--always in parent reference frame-->
     <!-- we have to rotate 45 around z to match the robotiq, while the robotiq has to rotate the same to match the real robot -->
@@ -112,5 +112,5 @@
     <!--<axis xyz="0 0 1" />-->
   </joint>
-  <link name="wrist_sr300_realsense_mount_link" >
+  <link name="wrist_camera_mount_link" >
     <inertial>
       <mass value="0.1"/>
@@ -140,5 +140,5 @@
   <!-- it is not determined by the xyzrpy in realsense.gazebo,xacro and realsense.urdf.xacro -->
   <!-- because everything inside realsense.gazebo,xacro and realsense.urdf.xacro are used for visualizing the camera. What the camera will see will not be influenced by its visualization parameters. -->
-  <xacro:property name="wrist_sr300_name" value="wrist_sr300_realsense" />
+  <xacro:property name="wrist_camera_name" value="wrist_camera" />
   <!--<xacro:property name="realsense_xyz" value="0.0 0.065 0.052"/>-->
   <xacro:property name="realsense_xyz" value="0.01 0.06 0.072"/>
@@ -147,31 +147,31 @@
   <!-- The rpy for simulation is different from the rpy setup for the actual camera. If we use the rpy from actual camera in simulation, the view will be wrong -->
   <!-- gazebo plug-in for simulating the camera -->
-  <xacro:if value="$(arg load_wrist_sr300_simulator)">
+  <xacro:if value="$(arg load_wrist_camera_simulator)">
     <xacro:realsense
-    sim="$(arg load_wrist_sr300_simulator)"
-    name="${wrist_sr300_name}"
-    parent="wrist_sr300_realsense_mount_link">
+    sim="$(arg load_wrist_camera_simulator)"
+    name="${wrist_camera_name}"
+    parent="wrist_camera_mount_link">
       <!-- <origin xyz="0.0 0.065 0.038" rpy="0.0 -${90/180*pi} -${90/180*pi}"/> -->
       <origin xyz="${realsense_xyz}" rpy="${realsense_rpy}"/>
     </xacro:realsense>
     <xacro:realsense_rgb_gazebo_v0
-    name="${wrist_sr300_name}"
-    link_name="${wrist_sr300_name}_rgb_frame"
-    frame_name="${wrist_sr300_name}_rgb_optical_frame"
-    camera_name="${wrist_sr300_name}"
-    visualize_wrist_sr300_simulator="$(arg visualize_wrist_sr300_simulator)" />
+    name="${wrist_camera_name}"
+    link_name="${wrist_camera_name}_rgb_frame"
+    frame_name="${wrist_camera_name}_rgb_optical_frame"
+    camera_name="${wrist_camera_name}"
+    visualize_wrist_camera_simulator="$(arg visualize_wrist_camera_simulator)" />
     <xacro:realsense_ir_gazebo_v0
-    name="${wrist_sr300_name}"
-    link_name="${wrist_sr300_name}_depth_frame"
-    frame_name="${wrist_sr300_name}_depth_optical_frame"
-    camera_name="${wrist_sr300_name}"
-    visualize_wrist_sr300_simulator="$(arg visualize_wrist_sr300_simulator)" />
+    name="${wrist_camera_name}"
+    link_name="${wrist_camera_name}_depth_frame"
+    frame_name="${wrist_camera_name}_depth_optical_frame"
+    camera_name="${wrist_camera_name}"
+    visualize_wrist_camera_simulator="$(arg visualize_wrist_camera_simulator)" />
   </xacro:if>
   <!-- if not in simulation: -->
-  <xacro:unless value="$(arg load_wrist_sr300_simulator)">
+  <xacro:unless value="$(arg load_wrist_camera_simulator)">
     <xacro:realsense
-    sim="$(arg load_wrist_sr300_simulator)"
-    name="${wrist_sr300_name}"
-    parent="wrist_sr300_realsense_mount_link">
+    sim="$(arg load_wrist_camera_simulator)"
+    name="${wrist_camera_name}"
+    parent="wrist_camera_mount_link">
       <!--<origin xyz="0. -0.25 0.5" rpy="0.0 0.0 -1.57"/>-->
       <origin xyz="${realsense_xyz}" rpy="${realsense_rpy}"/>

Commit message: switch r200

File: cob_hardware_config/robots/raw3-6/urdf/raw3-6.urdf.xacro (robot description, xacro)
@@ -43,5 +43,5 @@
     <origin xyz="${arm_x} ${arm_y} ${arm_z}" rpy="${arm_roll} ${arm_pitch} ${arm_yaw}" />
   </xacro:ur10>
-  <!--directlt defined here instead of retrieving from-->
+  <!--Directly defined here instead of retrieving from-->
   <!--$(find cob_hardware_config)/robots/raw3-6/urdf/properties.urdf.xacro-->
   <!--it has to be arm_tool0 instead of arm_ee_link-->
@@ -53,96 +53,11 @@
     <!-- We have to rotate the gripper by 45 around z, so that it matches the real robot -->
     <origin xyz="0 0 .05" rpy="${90/180*pi} 0 -${45/180*pi}"/>
-    <!--<origin xyz="0 0 .05" rpy="${90/180*pi} 0 -1.570795"/>-->
   </xacro:robotiq>
-  <!-- >>>>>>>>>>>>>>>>>>>>>>>>>>>>>>>>>>>>>>>>>>>>>>>>>>>>>>>>>>>>>>>>>> -->
-  <!-- wrist_camera mount and camera -->
-  <!--we add the sensor above the robot base metal board-->
-  <!--x = in the middle of the base metal board-->
-  <!--z = as high as the arm shoulder square base-->
-  <!--y = in the middle of the 2 batteries under the base metal board-->
-  <!--z - blue axis - larger is going up-->
-  <!--x - red axis - larger is going forward the robot-->
-  <!--y - green axis - larger is going left to robot-->
-  <!--yaw - rotate around z, 1.57 is 90 degree, so the camera is facing to the right-->
-<!--  <joint name="wrist_camera_mount_joint" type="fixed">-->
-    <!--[><xacro:insert_block name="origin" /><]-->
-    <!--<parent link="arm_tool0"/>-->
-    <!--<child link="wrist_camera_mount_link"/>-->
-    <!--[>always in parent reference frame<]-->
-    <!--[> we have to rotate 45 around z to match the robotiq, while the robotiq has to rotate the same to match the real robot <]-->
-    <!--<origin xyz="0.05 0.065 0.0025" rpy="0 0 -${45/180*pi}" />-->
-    <!--[> <origin xyz="0.0 0.075 0.0025" rpy="0 0 0" /> <]-->
-    <!--[>for prismatic and revolute (in local joint reference frame)<]-->
-    <!--[><axis xyz="0 0 1" /><]-->
-  <!--</joint>-->
-  <!--<link name="wrist_camera_mount_link" >-->
-    <!--<inertial>-->
-      <!--<mass value="0.1"/>-->
-      <!--<origin xyz="0 0 0"/>-->
-      <!--[>https://gist.github.com/awesomebytes/39a4ba6c64956a1aa9bd<]-->
-      <!--<inertia ixx="0.00018" ixy="0.0" ixz="0.0" iyy="0.00002" iyz="0.0" izz="0.0002" />-->
-    <!--</inertial>-->
-    <!--<visual>-->
-      <!--<origin xyz="0.0 0.0 0.0" rpy="0 0 0"/>-->
-      <!--<geometry>-->
-        <!--<box size="0.05 0.150 0.005"/>-->
-      <!--</geometry>-->
-      <!--<material name="gray">-->
-        <!--<color rgba="0.50 0.50 0.50 1" />-->
-        <!--[> <color rgba="1.0 1.0 1.0 1" /> <]-->
-        <!--[><color rgba="0.2 0.2 1 1" /><]-->
-      <!--</material>-->
-    <!--</visual>-->
-    <!--<collision>-->
-      <!--<origin xyz="0.0 0.0 0.0" rpy="0 0 0"/>-->
-      <!--<geometry>-->
-        <!--<box size="0.05 0.150 0.005"/>-->
-      <!--</geometry>-->
-    <!--</collision>-->
-  <!--</link>-->
-  <joint name="wrist_camera_mount_joint" type="fixed">
-    <!--<xacro:insert_block name="origin" />-->
-    <parent link="gripper_palm"/>
-    <child link="wrist_camera_mount_link"/>
-    <!--always in parent reference frame-->
-    <!-- we have to rotate 45 around z to match the robotiq, while the robotiq has to rotate the same to match the real robot -->
-    <origin xyz="0.00 -0.02 -0.05" rpy="-${90/180*pi} 0 0" />
-    <!-- <origin xyz="0.0 0.075 0.0025" rpy="0 0 0" /> -->
-    <!--for prismatic and revolute (in local joint reference frame)-->
-    <!--<axis xyz="0 0 1" />-->
-  </joint>
-  <link name="wrist_camera_mount_link" >
-    <inertial>
-      <mass value="0.1"/>
-      <origin xyz="0 0 0"/>
-      <!--https://gist.github.com/awesomebytes/39a4ba6c64956a1aa9bd-->
-      <inertia ixx="0.00018" ixy="0.0" ixz="0.0" iyy="0.00002" iyz="0.0" izz="0.0002" />
-    </inertial>
-    <visual>
-      <origin xyz="0.0 0.0 0.0" rpy="0 0 0"/>
-      <geometry>
-        <box size="0.05 0.08 0.005"/>
-      </geometry>
-      <material name="gray">
-        <color rgba="0.50 0.50 0.50 1" />
-        <!-- <color rgba="1.0 1.0 1.0 1" /> -->
-        <!--<color rgba="0.2 0.2 1 1" />-->
-      </material>
-    </visual>
-    <collision>
-      <origin xyz="0.0 0.0 0.0" rpy="0 0 0"/>
-      <geometry>
-        <box size="0.05 0.08 0.005"/>
-      </geometry>
-    </collision>
-  </link>
   <!-- the view of the camera is only determined by the following xyzrpy -->
   <!-- it is not determined by the xyzrpy in realsense.gazebo,xacro and realsense.urdf.xacro -->
   <!-- because everything inside realsense.gazebo,xacro and realsense.urdf.xacro are used for visualizing the camera. What the camera will see will not be influenced by its visualization parameters. -->
   <xacro:property name="wrist_camera_name" value="wrist_camera" />
-  <!--<xacro:property name="realsense_xyz" value="0.0 0.065 0.052"/>-->
-  <xacro:property name="realsense_xyz" value="0.01 0.06 0.072"/>
-  <!--<xacro:property name="realsense_rpy" value="0.0 0.0 ${180/180*pi}"/>-->
-  <xacro:property name="realsense_rpy" value="0.0 0.0 ${180/180*pi}"/>
+  <xacro:property name="realsense_xyz" value="-0.0381 0.0127 -0.0762"/>
+  <xacro:property name="realsense_rpy" value="-${90/180*pi} 0.0 0.0"/>
   <!-- The rpy for simulation is different from the rpy setup for the actual camera. If we use the rpy from actual camera in simulation, the view will be wrong -->
   <!-- gazebo plug-in for simulating the camera -->
@@ -151,6 +66,5 @@
     sim="$(arg load_wrist_camera_simulator)"
     name="${wrist_camera_name}"
-    parent="wrist_camera_mount_link">
-      <!-- <origin xyz="0.0 0.065 0.038" rpy="0.0 -${90/180*pi} -${90/180*pi}"/> -->
+    parent="gripper_palm">
       <origin xyz="${realsense_xyz}" rpy="${realsense_rpy}"/>
     </xacro:realsense>
@@ -173,6 +87,5 @@
     sim="$(arg load_wrist_camera_simulator)"
     name="${wrist_camera_name}"
-    parent="wrist_camera_mount_link">
-      <!--<origin xyz="0. -0.25 0.5" rpy="0.0 0.0 -1.57"/>-->
+    parent="gripper_palm">
       <origin xyz="${realsense_xyz}" rpy="${realsense_rpy}"/>
     </xacro:realsense>

Commit message: switch r200

File: cob_hardware_config/robots/raw3-6/urdf/raw3-6.urdf.xacro (robot description, xacro)
@@ -59,5 +59,5 @@
   <xacro:property name="wrist_camera_name" value="wrist_camera" />
   <xacro:property name="realsense_xyz" value="-0.0381 0.0127 -0.0762"/>
-  <xacro:property name="realsense_rpy" value="-${90/180*pi} 0.0 0.0"/>
+  <xacro:property name="realsense_rpy" value="-${90/180*pi} ${180/180*pi} 0.0"/>
   <!-- The rpy for simulation is different from the rpy setup for the actual camera. If we use the rpy from actual camera in simulation, the view will be wrong -->
   <!-- gazebo plug-in for simulating the camera -->

Commit message: change r200 pos

File: cob_hardware_config/robots/raw3-6/urdf/raw3-6.urdf.xacro (robot description, xacro)
@@ -58,5 +58,5 @@
   <!-- because everything inside realsense.gazebo,xacro and realsense.urdf.xacro are used for visualizing the camera. What the camera will see will not be influenced by its visualization parameters. -->
   <xacro:property name="wrist_camera_name" value="wrist_camera" />
-  <xacro:property name="realsense_xyz" value="-0.0381 0.0127 -0.0762"/>
+  <xacro:property name="realsense_xyz" value="-0.0481 0.0027 -0.0762"/>
   <xacro:property name="realsense_rpy" value="-${90/180*pi} ${180/180*pi} 0.0"/>
   <!-- The rpy for simulation is different from the rpy setup for the actual camera. If we use the rpy from actual camera in simulation, the view will be wrong -->

Commit message: fix transformation bw r200 and palm, lens and r200 via compute-obj2obj in yuripy, refactor realsense -> r200

File: cob_hardware_config/robots/raw3-6/urdf/raw3-6.urdf.xacro (robot description, xacro)
@@ -18,8 +18,7 @@
   <!-- robotiq gripper -->
   <xacro:include filename="$(find cob_description)/urdf/robotiq_gripper/robotiq_s_gripper.urdf.xacro" />
-  <!-- RealSense Sensors -->
-  <!--<xacro:include filename="$(find cob_description)/urdf/sensors/r200.urdf.xacro"/>-->
-  <xacro:include filename="$(find cob_description)/urdf/sensors/realsense.urdf.xacro"/>
-  <xacro:include filename="$(find cob_description)/urdf/sensors/realsense.gazebo.xacro"/>
+  <!-- r200 Sensors -->
+  <xacro:include filename="$(find cob_description)/urdf/sensors/r200.urdf.xacro"/>
+  <xacro:include filename="$(find cob_description)/urdf/sensors/r200.gazebo.xacro"/>
   <!-- sick s300 -->
   <xacro:include filename="$(find cob_description)/urdf/sensors/sick_s300_laser.urdf.xacro"/>
@@ -54,20 +53,18 @@
     <origin xyz="0 0 .05" rpy="${90/180*pi} 0 -${45/180*pi}"/>
   </xacro:robotiq>
-  <!-- the view of the camera is only determined by the following xyzrpy -->
-  <!-- it is not determined by the xyzrpy in realsense.gazebo,xacro and realsense.urdf.xacro -->
-  <!-- because everything inside realsense.gazebo,xacro and realsense.urdf.xacro are used for visualizing the camera. What the camera will see will not be influenced by its visualization parameters. -->
   <xacro:property name="wrist_camera_name" value="wrist_camera" />
-  <xacro:property name="realsense_xyz" value="-0.0481 0.0027 -0.0762"/>
-  <xacro:property name="realsense_rpy" value="-${90/180*pi} ${180/180*pi} 0.0"/>
+  <!-- wrist_camera_r200_xyz and wrist_camera_r200_rpy = r200_in_palm_mat -->
+  <xacro:property name="wrist_camera_r200_xyz" value="0.0057  0.0012 -0.0746"/>
+  <xacro:property name="wrist_camera_r200_rpy" value="0 1.57 1.57"/>
   <!-- The rpy for simulation is different from the rpy setup for the actual camera. If we use the rpy from actual camera in simulation, the view will be wrong -->
   <!-- gazebo plug-in for simulating the camera -->
   <xacro:if value="$(arg load_wrist_camera_simulator)">
-    <xacro:realsense
+    <xacro:r200
     sim="$(arg load_wrist_camera_simulator)"
     name="${wrist_camera_name}"
     parent="gripper_palm">
-      <origin xyz="${realsense_xyz}" rpy="${realsense_rpy}"/>
-    </xacro:realsense>
-    <xacro:realsense_rgb_gazebo_v0
+      <origin xyz="${wrist_camera_r200_xyz}" rpy="${wrist_camera_r200_rpy}"/>
+    </xacro:r200>
+    <xacro:r200_rgb_gazebo_v0
     name="${wrist_camera_name}"
     link_name="${wrist_camera_name}_rgb_frame"
@@ -75,5 +72,5 @@
     camera_name="${wrist_camera_name}"
     visualize_wrist_camera_simulator="$(arg visualize_wrist_camera_simulator)" />
-    <xacro:realsense_ir_gazebo_v0
+    <xacro:r200_ir_gazebo_v0
     name="${wrist_camera_name}"
     link_name="${wrist_camera_name}_depth_frame"
@@ -84,10 +81,10 @@
   <!-- if not in simulation: -->
   <xacro:unless value="$(arg load_wrist_camera_simulator)">
-    <xacro:realsense
+    <xacro:r200
     sim="$(arg load_wrist_camera_simulator)"
     name="${wrist_camera_name}"
     parent="gripper_palm">
-      <origin xyz="${realsense_xyz}" rpy="${realsense_rpy}"/>
-    </xacro:realsense>
+      <origin xyz="${wrist_camera_r200_xyz}" rpy="${wrist_camera_r200_rpy}"/>
+    </xacro:r200>
   </xacro:unless>
   <!--
