Commit message: fix r200 pos

File: cob_hardware_config/robots/raw3-6/urdf/raw3-6.urdf.xacro (robot description, xacro)
@@ -55,5 +55,5 @@
   <xacro:property name="wrist_camera_name" value="wrist_camera" />
   <!-- wrist_camera_r200_xyz and wrist_camera_r200_rpy = r200_in_palm_mat -->
-  <xacro:property name="wrist_camera_r200_xyz" value="0.0057  0.0012 -0.0746"/>
+  <xacro:property name="wrist_camera_r200_xyz" value="-0.0057  0.0012 -0.0746"/>
   <xacro:property name="wrist_camera_r200_rpy" value="0 1.57 1.57"/>
   <!-- The rpy for simulation is different from the rpy setup for the actual camera. If we use the rpy from actual camera in simulation, the view will be wrong -->

Commit message: add frame for sensor

File: cob_hardware_config/robots/raw3-6/urdf/raw3-6.urdf.xacro (robot description, xacro)
@@ -55,5 +55,8 @@
   <xacro:property name="wrist_camera_name" value="wrist_camera" />
   <!-- wrist_camera_r200_xyz and wrist_camera_r200_rpy = r200_in_palm_mat -->
-  <xacro:property name="wrist_camera_r200_xyz" value="-0.0057  0.0012 -0.0746"/>
+  <!-- z - up or down on the gripper -->
+  <!-- y - front or back from the gripper -->
+  <!-- x - left or right side from the gripper -->
+  <xacro:property name="wrist_camera_r200_xyz" value="0.0157  0.0012 -0.1006"/>
   <xacro:property name="wrist_camera_r200_rpy" value="0 1.57 1.57"/>
   <!-- The rpy for simulation is different from the rpy setup for the actual camera. If we use the rpy from actual camera in simulation, the view will be wrong -->
@@ -88,4 +91,28 @@
     </xacro:r200>
   </xacro:unless>
+  <joint name="${wrist_camera_name}_mount_joint" type="fixed">
+    <origin xyz="-0.01 -0.012 -0.03" rpy="0 0 0" />
+    <parent link="${wrist_camera_name}_link"/>
+    <child link="${wrist_camera_name}_mount_link"/>
+  </joint>
+  <link name="${wrist_camera_name}_mount_link" >
+    <inertial>
+      <mass value="0.564" />
+      <origin xyz="0.0 0.0 0.0" rpy="0.0 0.0 0.0" />
+      <inertia ixx="0.003881243" ixy="0.0" ixz="0.0" iyy="0.000498940" iyz="0.0" izz="0.003879257" />
+    </inertial>
+    <visual>
+     <origin xyz="0.0 0.0 0.0" rpy="0.0 0.0 0.0"/>
+      <geometry>
+        <box size="0.04 0.15 0.05"/>
+      </geometry>
+    </visual>
+    <collision>
+     <origin xyz="0.0 0.0 0.0" rpy="0.0 0.0 0.0"/>
+      <geometry>
+        <box size="0.04 0.15 0.05"/>
+      </geometry>
+    </collision>
+  </link>
   <!--
   <xacro:sensor_r200 prefix="vision_wrist_" parent="arm_tool0">

Commit message: add sim camera to real run also

File: cob_hardware_config/robots/raw3-6/urdf/raw3-6.urdf.xacro (robot description, xacro)
@@ -62,12 +62,13 @@
   <!-- The rpy for simulation is different from the rpy setup for the actual camera. If we use the rpy from actual camera in simulation, the view will be wrong -->
   <!-- gazebo plug-in for simulating the camera -->
+  <xacro:r200
+  sim="$(arg load_wrist_camera_simulator)"
+  name="${wrist_camera_name}"
+  parent="gripper_palm">
+    <origin xyz="${wrist_camera_r200_xyz}" rpy="${wrist_camera_r200_rpy}"/>
+  </xacro:r200>
   <xacro:if value="$(arg load_wrist_camera_simulator)">
-    <xacro:r200
+    <xacro:r200_rgb_gazebo_v0
     sim="$(arg load_wrist_camera_simulator)"
-    name="${wrist_camera_name}"
-    parent="gripper_palm">
-      <origin xyz="${wrist_camera_r200_xyz}" rpy="${wrist_camera_r200_rpy}"/>
-    </xacro:r200>
-    <xacro:r200_rgb_gazebo_v0
     name="${wrist_camera_name}"
     link_name="${wrist_camera_name}_rgb_frame"
@@ -76,4 +77,5 @@
     visualize_wrist_camera_simulator="$(arg visualize_wrist_camera_simulator)" />
     <xacro:r200_ir_gazebo_v0
+    sim="$(arg load_wrist_camera_simulator)"
     name="${wrist_camera_name}"
     link_name="${wrist_camera_name}_depth_frame"
@@ -82,13 +84,4 @@
     visualize_wrist_camera_simulator="$(arg visualize_wrist_camera_simulator)" />
   </xacro:if>
-  <!-- if not in simulation: -->
-  <xacro:unless value="$(arg load_wrist_camera_simulator)">
-    <xacro:r200
-    sim="$(arg load_wrist_camera_simulator)"
-    name="${wrist_camera_name}"
-    parent="gripper_palm">
-      <origin xyz="${wrist_camera_r200_xyz}" rpy="${wrist_camera_r200_rpy}"/>
-    </xacro:r200>
-  </xacro:unless>
   <joint name="${wrist_camera_name}_mount_joint" type="fixed">
     <origin xyz="-0.01 -0.012 -0.03" rpy="0 0 0" />

Commit message: reduce mesh for camera, so that insertion pose 3 in lm works

File: cob_hardware_config/robots/raw3-6/urdf/raw3-6.urdf.xacro (robot description, xacro)
@@ -90,4 +90,5 @@
     <child link="${wrist_camera_name}_mount_link"/>
   </joint>
+  <!-- The collisions for the mount link is  used for [despot_motion](https://github.com/Shentheman/despot_motion) -->
   <link name="${wrist_camera_name}_mount_link" >
     <inertial>
@@ -99,5 +100,6 @@
      <origin xyz="0.0 0.0 0.0" rpy="0.0 0.0 0.0"/>
       <geometry>
-        <box size="0.04 0.15 0.05"/>
+        <!-- <box size="0.04 0.15 0.05"/> -->
+        <box size="0.05 0.05 0.05"/>
       </geometry>
     </visual>
@@ -105,5 +107,6 @@
      <origin xyz="0.0 0.0 0.0" rpy="0.0 0.0 0.0"/>
       <geometry>
-        <box size="0.04 0.15 0.05"/>
+        <!-- <box size="0.04 0.15 0.05"/> -->
+        <box size="0.05 0.05 0.05"/>
       </geometry>
     </collision>

Commit message: udpate ik solver and camera collision model to be smaller

File: cob_hardware_config/robots/raw3-6/urdf/raw3-6.urdf.xacro (robot description, xacro)
@@ -98,5 +98,6 @@
      <origin xyz="0.0 0.0 0.0" rpy="0.0 0.0 0.0"/>
       <geometry>
-        <box size="0.04 0.15 0.05"/>
+        <!-- <box size="0.04 0.15 0.05"/> -->
+        <box size="0.05 0.05 0.05"/>
       </geometry>
     </visual>
@@ -104,5 +105,6 @@
      <origin xyz="0.0 0.0 0.0" rpy="0.0 0.0 0.0"/>
       <geometry>
-        <box size="0.04 0.15 0.05"/>
+        <!-- <box size="0.04 0.15 0.05"/> -->
+        <box size="0.05 0.05 0.05"/>
       </geometry>
     </collision>

Commit message: add option to fix base

File: cob_hardware_config/robots/raw3-6/urdf/raw3-6.urdf.xacro (robot description, xacro)
@@ -3,4 +3,5 @@
        name="raw3-6" >
   <arg name="load_wrist_camera_simulator" default="$(optenv LOAD_WRIST_CAMERA_SIMULATOR !!NO_LOAD_WRIST_CAMERA_SIMULATOR_SET!!)"/>
+  <arg name="fix_base_with_world" default="$(optenv FIX_BASE_WITH_WORLD !!NO_FIX_BASE_WITH_WORLD_SET!!)"/>
   <arg name="visualize_wrist_camera_simulator" default="$(optenv VISUALIZE_WRIST_CAMERA_SIMULATOR !!NO_VISUALIZE_WRIST_CAMERA_SIMULATOR_SET!!)"/>
   <arg name="visualize_sick_s300_simulator" default="$(optenv VISUALIZE_SICK_S300_SIMULATOR !!NO_VISUALIZE_SICK_S300_SIMULATOR_SET!!)"/>
@@ -26,5 +27,6 @@
   <xacro:include filename="$(find cob_description)/urdf/sensors/sick_s300_laser.urdf.xacro"/>
   <!-- composition of the robot -->
-  <xacro:raw_base sim="$(arg sim)" visualize_sick_s300_simulator="$(arg visualize_sick_s300_simulator)" name="base"/>
+  <xacro:property name="base_name" value="base" />
+  <xacro:raw_base sim="$(arg sim)" visualize_sick_s300_simulator="$(arg visualize_sick_s300_simulator)" name="${base_name}"/>
   <!-- These are already defined at ./src/cob_common/raw_description/urdf/base_long/base.urdf.xacro. -->
   <!-- These are already defined at ./src/cob_common/raw_description/urdf/base_short/base.urdf.xacro. -->
@@ -110,4 +112,14 @@
     </collision>
   </link>
+  <!-- If we don't want the base to move at all: -->
+  <!-- https://github.com/ros-industrial/universal_robot/blob/830a7b480063d66b22d939c42a0c6c08901713e6/ur_description/urdf/ur10_joint_limited_robot.urdf.xacro#L21 -->
+  <xacro:if value="$(arg fix_base_with_world)">
+    <link name="world" />
+    <joint name="world_joint" type="fixed">
+      <parent link="world" />
+      <child link = "${base_name}_footprint" />
+      <origin xyz="0.0 0.0 0.0" rpy="0.0 0.0 0.0" />
+    </joint>
+  </xacro:if>
   <!--
   <xacro:sensor_r200 prefix="vision_wrist_" parent="arm_tool0">
