Commit message: make gazebo+moveit work for ur10

File: cob_hardware_config/robots/cob4-10/urdf/cob4-10.urdf.xacro (robot description, xacro)
@@ -5,4 +5,5 @@
   <xacro:include filename="$(find cob_description)/urdf/common.xacro" />
   <xacro:include filename="$(find cob_description)/urdf/materials.urdf.xacro" />
+  <xacro:include filename="$(find schunk_description)/urdf/materials.urdf.xacro" />
   <!-- calibration -->
   <xacro:include filename="$(find cob_hardware_config)/robots/cob4-10/urdf/properties.urdf.xacro" />

File: cob_hardware_config/robots/cob4-11/urdf/cob4-11.urdf.xacro (robot description, xacro)
@@ -5,4 +5,5 @@
   <xacro:include filename="$(find cob_description)/urdf/common.xacro" />
   <xacro:include filename="$(find cob_description)/urdf/materials.urdf.xacro" />
+  <xacro:include filename="$(find schunk_description)/urdf/materials.urdf.xacro" />
   <!-- calibration -->
   <xacro:include filename="$(find cob_hardware_config)/robots/cob4-11/urdf/properties.urdf.xacro" />

File: cob_hardware_config/robots/cob4-2/urdf/cob4-2.urdf.xacro (robot description, xacro)
@@ -5,4 +5,5 @@
   <xacro:include filename="$(find cob_description)/urdf/common.xacro" />
   <xacro:include filename="$(find cob_description)/urdf/materials.urdf.xacro" />
+  <xacro:include filename="$(find schunk_description)/urdf/materials.urdf.xacro" />
   <!-- calibration -->
   <xacro:include filename="$(find cob_hardware_config)/robots/cob4-2/urdf/properties.urdf.xacro" />

File: cob_hardware_config/robots/cob4-5/urdf/cob4-5.urdf.xacro (robot description, xacro)
@@ -5,4 +5,5 @@
   <xacro:include filename="$(find cob_description)/urdf/common.xacro" />
   <xacro:include filename="$(find cob_description)/urdf/materials.urdf.xacro" />
+  <xacro:include filename="$(find schunk_description)/urdf/materials.urdf.xacro" />
   <!-- calibration -->
   <xacro:include filename="$(find cob_hardware_config)/robots/cob4-5/urdf/properties.urdf.xacro" />
@@ -12,5 +13,5 @@
   <xacro:include filename="$(find cob_description)/urdf/cob4_torso/torso.urdf.xacro" />
   <!-- arm -->
-  <xacro:include filename="$(find cob_description)/urdf/cob4_arm/cob4_arm.urdf.xacro" />
+  <xacro:include filename="$(find schunk_description)/urdf/lwa4p_extended/lwa4p_extended.urdf.xacro" />
   <!-- hand -->
   <xacro:include filename="$(find cob_description)/urdf/cob4_gripper/gripper.urdf.xacro" />
@@ -68,10 +69,10 @@
     <origin xyz="${sensorring_cam3d_back_x} ${sensorring_cam3d_back_y} ${sensorring_cam3d_back_z}" rpy="${sensorring_cam3d_back_roll} ${sensorring_cam3d_back_pitch} ${sensorring_cam3d_back_yaw}" />
   </xacro:cob_kinect_v0>
-  <xacro:cob4_arm name="arm_right" parent="torso_3_link" has_podest="false">
+  <xacro:schunk_lwa4p_extended name="arm_right" parent="torso_3_link" has_podest="false">
     <origin xyz="${arm_right_x} ${arm_right_y} ${arm_right_z}" rpy="${arm_right_roll} ${arm_right_pitch} ${arm_right_yaw}" />
-  </xacro:cob4_arm>
-  <xacro:cob4_arm name="arm_left" parent="torso_3_link" has_podest="false">
+  </xacro:schunk_lwa4p_extended>
+  <xacro:schunk_lwa4p_extended name="arm_left" parent="torso_3_link" has_podest="false">
     <origin xyz="${arm_left_x} ${arm_left_y} ${arm_left_z}" rpy="${arm_left_roll} ${arm_left_pitch} ${arm_left_yaw}" />
-  </xacro:cob4_arm>
+  </xacro:schunk_lwa4p_extended>
   <xacro:gripper name="gripper_right" parent="arm_right_7_link">
     <origin xyz="${gripper_right_x} ${gripper_right_y} ${gripper_right_z}" rpy="${gripper_right_roll} ${gripper_right_pitch} ${gripper_right_yaw}" />

File: cob_hardware_config/robots/cob4-7/urdf/cob4-7.urdf.xacro (robot description, xacro)
@@ -5,4 +5,5 @@
   <xacro:include filename="$(find cob_description)/urdf/common.xacro" />
   <xacro:include filename="$(find cob_description)/urdf/materials.urdf.xacro" />
+  <xacro:include filename="$(find schunk_description)/urdf/materials.urdf.xacro" />
   <!-- calibration -->
   <xacro:include filename="$(find cob_hardware_config)/robots/cob4-7/urdf/properties.urdf.xacro" />

File: cob_hardware_config/robots/cob4-8/urdf/cob4-8.urdf.xacro (robot description, xacro)
@@ -5,4 +5,5 @@
   <xacro:include filename="$(find cob_description)/urdf/common.xacro" />
   <xacro:include filename="$(find cob_description)/urdf/materials.urdf.xacro" />
+  <xacro:include filename="$(find schunk_description)/urdf/materials.urdf.xacro" />
   <!-- calibration -->
   <xacro:include filename="$(find cob_hardware_config)/robots/cob4-8/urdf/properties.urdf.xacro" />
@@ -12,5 +13,5 @@
   <xacro:include filename="$(find cob_description)/urdf/cob4_torso/torso.urdf.xacro" />
   <!-- arm -->
-  <xacro:include filename="$(find cob_description)/urdf/cob4_arm/cob4_arm.urdf.xacro" />
+  <xacro:include filename="$(find schunk_description)/urdf/lwa4p_extended/lwa4p_extended.urdf.xacro" />
   <!-- hand -->
   <xacro:include filename="$(find cob_description)/urdf/cob4_gripper/gripper.urdf.xacro" />
@@ -23,4 +24,5 @@
   <xacro:include filename="$(find cob_description)/urdf/sensors/kinect.urdf.xacro" />
   <xacro:include filename="$(find cob_description)/urdf/sensors/usb_cam.urdf.xacro" />
+  <xacro:include filename="$(find cob_description)/urdf/sensors/sick_3dcs.urdf.xacro" />
   <xacro:include filename="$(find cob_description)/urdf/sensors/sick_s300_laser.urdf.xacro"/>
   <!-- composition of the robot -->
@@ -64,10 +66,10 @@
     <origin xyz="${sensorring_cam3d_x} ${sensorring_cam3d_y} ${sensorring_cam3d_z}" rpy="${sensorring_cam3d_roll} ${sensorring_cam3d_pitch} ${sensorring_cam3d_yaw}" />
   </xacro:cob_kinect_v0>
-  <xacro:cob4_arm name="arm_right" parent="torso_3_link" has_podest="false">
+  <xacro:schunk_lwa4p_extended name="arm_right" parent="torso_3_link" has_podest="false">
     <origin xyz="${arm_right_x} ${arm_right_y} ${arm_right_z}" rpy="${arm_right_roll} ${arm_right_pitch} ${arm_right_yaw}" />
-  </xacro:cob4_arm>
-  <xacro:cob4_arm name="arm_left" parent="torso_3_link" has_podest="false">
+  </xacro:schunk_lwa4p_extended>
+  <xacro:schunk_lwa4p_extended name="arm_left" parent="torso_3_link" has_podest="false">
     <origin xyz="${arm_left_x} ${arm_left_y} ${arm_left_z}" rpy="${arm_left_roll} ${arm_left_pitch} ${arm_left_yaw}" />
-  </xacro:cob4_arm>
+  </xacro:schunk_lwa4p_extended>
   <xacro:gripper name="gripper_right" parent="arm_right_7_link">
     <origin xyz="${gripper_right_x} ${gripper_right_y} ${gripper_right_z}" rpy="${gripper_right_roll} ${gripper_right_pitch} ${gripper_right_yaw}" />

File: cob_hardware_config/robots/cob4-9/urdf/cob4-9.urdf.xacro (robot description, xacro)
@@ -5,4 +5,5 @@
   <xacro:include filename="$(find cob_description)/urdf/common.xacro" />
   <xacro:include filename="$(find cob_description)/urdf/materials.urdf.xacro" />
+  <xacro:include filename="$(find schunk_description)/urdf/materials.urdf.xacro" />
   <!-- calibration -->
   <xacro:include filename="$(find cob_hardware_config)/robots/cob4-9/urdf/properties.urdf.xacro" />

File: cob_hardware_config/robots/raw3-1/urdf/raw3-1.urdf.xacro (robot description, xacro)
@@ -15,5 +15,5 @@
   <xacro:include filename="$(find raw_description)/urdf/head/head.urdf.xacro" />
   <!-- ur_arm -->
-  <xacro:include filename="$(find raw_description)/urdf/ur_arm/ur10_arm.urdf.xacro" />
+  <xacro:include filename="$(find cob_description)/urdf/ur_arm/ur10_arm.urdf.xacro" />
   <!-- vacuum gripper -->
   <xacro:include filename="$(find raw_description)/urdf/vacuum_gripper/gripper.urdf.xacro" />

File: cob_hardware_config/robots/raw3-6/urdf/calibration_default.urdf.xacro (robot description, xacro)
@@ -1,37 +1,45 @@
 <?xml version="1.0"?>
-<robot>
+<robot xmlns:xacro="http://www.ros.org/wiki/xacro">
 	<!-- ***************** -->
 	<!-- base calibration -->
 	<!-- ***************** -->
 	<!-- laser front mount positions | relative to base_link -->
-	<property name="def_laser_front_x" value="0.465"/>
-	<property name="def_laser_front_y" value="-0.232"/>
-	<property name="def_laser_front_z" value="0.178"/>
-	<property name="def_laser_front_roll" value="${M_PI}"/>
-	<property name="def_laser_front_pitch" value="0.0"/>
-	<property name="def_laser_front_yaw" value="${-M_PI/4}"/>
+	<xacro:property name="def_laser_front_x" value="0.465"/>
+	<xacro:property name="def_laser_front_y" value="-0.232"/>
+	<xacro:property name="def_laser_front_z" value="0.178"/>
+	<xacro:property name="def_laser_front_roll" value="${M_PI}"/>
+	<xacro:property name="def_laser_front_pitch" value="0.0"/>
+	<xacro:property name="def_laser_front_yaw" value="${-M_PI/4}"/>
 	<!-- laser rear mount positions | relative to base_link -->
-	<property name="def_laser_rear_x" value="-0.465"/>
-	<property name="def_laser_rear_y" value="0.232"/>
-	<property name="def_laser_rear_z" value="0.178"/>
-	<property name="def_laser_rear_roll" value="${M_PI}"/>
-	<property name="def_laser_rear_pitch" value="0.0"/>
-	<property name="def_laser_rear_yaw" value="${-5*M_PI/4}"/>
-	<!-- *********************************** -->
-	<!-- kinematic chain reference positions -->
-	<!-- *********************************** -->
+	<xacro:property name="def_laser_rear_x" value="-0.465"/>
+	<xacro:property name="def_laser_rear_y" value="0.232"/>
+	<xacro:property name="def_laser_rear_z" value="0.178"/>
+	<xacro:property name="def_laser_rear_roll" value="${M_PI}"/>
+	<xacro:property name="def_laser_rear_pitch" value="0.0"/>
+	<xacro:property name="def_laser_rear_yaw" value="${-5*M_PI/4}"/>
+    <!-- *********************************** -->
+    <!-- kinematic chain reference positions -->
+    <!-- *********************************** -->
 	<!-- tower mount positions | relative to base_link -->
-	<property name="def_tower_x" value="0.361"/>
-	<property name="def_tower_y" value="0.0"/>
-	<property name="def_tower_z" value="0.306"/>
-	<property name="def_tower_roll" value="0.0"/>
-	<property name="def_tower_pitch" value="0.0"/>
-	<property name="def_tower_yaw" value="0.0"/>
+	<xacro:property name="def_tower_x" value="0.361"/>
+	<xacro:property name="def_tower_y" value="0.0"/>
+	<xacro:property name="def_tower_z" value="0.306"/>
+	<xacro:property name="def_tower_roll" value="0.0"/>
+	<xacro:property name="def_tower_pitch" value="0.0"/>
+	<xacro:property name="def_tower_yaw" value="0.0"/>
 	<!--arm mount positions | relative to base_link-->
-	<property name="def_arm_x" value="0.330"/>
-	<property name="def_arm_y" value="0.0"/>
-	<property name="def_arm_z" value="0.482"/>
-	<property name="def_arm_roll" value="0.0"/>
-	<property name="def_arm_pitch" value="0.0"/>
-	<property name="def_arm_yaw" value="${-M_PI/2}"/>
+	<xacro:property name="def_arm_x" value="0.330"/>
+	<xacro:property name="def_arm_y" value="0.0"/>
+	<xacro:property name="def_arm_z" value="0.482"/>
+	<xacro:property name="def_arm_roll" value="0.0"/>
+	<xacro:property name="def_arm_pitch" value="0.0"/>
+	<xacro:property name="def_arm_yaw" value="${-M_PI/2}"/>
+	<!-- gripper mount positions | relative to arm_ee_link -->
+    <!--directly defined at ./src/cob_robots/cob_hardware_config/robots/raw3-6/urdf/raw3-6.urdf.xacro-->
+	<!--<xacro:property name="def_gripper_x" value="0.0"/>-->
+	<!--<xacro:property name="def_gripper_y" value="0.0"/>-->
+	<!--<xacro:property name="def_gripper_z" value="0.0"/>-->
+	<!--<xacro:property name="def_gripper_roll" value="0.0"/>-->
+	<!--<xacro:property name="def_gripper_pitch" value="0.0"/>-->
+	<!--<xacro:property name="def_gripper_yaw" value="0.0"/>-->
 </robot>

File: cob_hardware_config/robots/raw3-6/urdf/properties.urdf.xacro (robot description, xacro)
@@ -8,33 +8,41 @@
 	<!-- laser front mount positions | relative to base_link -->
     <!--XXX: these parameters e.g. def_laser_front_x are from cob_robots/cob_hardware_config/robots/raw3-5/urdf/calibration_default.urdf.xacro-->
-	<property name="laser_front_x" value="${def_laser_front_x+offset_laser_front_x}"/>
-	<property name="laser_front_y" value="${def_laser_front_y+offset_laser_front_y}"/>
-	<property name="laser_front_z" value="${def_laser_front_z+offset_laser_front_z}"/>
-	<property name="laser_front_roll" value="${def_laser_front_roll+offset_laser_front_roll}"/>
-	<property name="laser_front_pitch" value="${def_laser_front_pitch+offset_laser_front_pitch}"/>
-	<property name="laser_front_yaw" value="${def_laser_front_yaw+offset_laser_front_yaw}"/>
+	<xacro:property name="laser_front_x" value="${def_laser_front_x+offset_laser_front_x}"/>
+	<xacro:property name="laser_front_y" value="${def_laser_front_y+offset_laser_front_y}"/>
+	<xacro:property name="laser_front_z" value="${def_laser_front_z+offset_laser_front_z}"/>
+	<xacro:property name="laser_front_roll" value="${def_laser_front_roll+offset_laser_front_roll}"/>
+	<xacro:property name="laser_front_pitch" value="${def_laser_front_pitch+offset_laser_front_pitch}"/>
+	<xacro:property name="laser_front_yaw" value="${def_laser_front_yaw+offset_laser_front_yaw}"/>
 	<!-- laser rear mount positions | relative to base_link -->
-	<property name="laser_rear_x" value="${def_laser_rear_x+offset_laser_rear_x}"/>
-	<property name="laser_rear_y" value="${def_laser_rear_y+offset_laser_rear_y}"/>
-	<property name="laser_rear_z" value="${def_laser_rear_z+offset_laser_rear_z}"/>
-	<property name="laser_rear_roll" value="${def_laser_rear_roll+offset_laser_rear_roll}"/>
-	<property name="laser_rear_pitch" value="${def_laser_rear_pitch+offset_laser_rear_pitch}"/>
-	<property name="laser_rear_yaw" value="${def_laser_rear_yaw+offset_laser_rear_yaw}"/>
+	<xacro:property name="laser_rear_x" value="${def_laser_rear_x+offset_laser_rear_x}"/>
+	<xacro:property name="laser_rear_y" value="${def_laser_rear_y+offset_laser_rear_y}"/>
+	<xacro:property name="laser_rear_z" value="${def_laser_rear_z+offset_laser_rear_z}"/>
+	<xacro:property name="laser_rear_roll" value="${def_laser_rear_roll+offset_laser_rear_roll}"/>
+	<xacro:property name="laser_rear_pitch" value="${def_laser_rear_pitch+offset_laser_rear_pitch}"/>
+	<xacro:property name="laser_rear_yaw" value="${def_laser_rear_yaw+offset_laser_rear_yaw}"/>
 	<!-- *********************** -->
 	<!-- upper robot calibration -->
 	<!-- *********************** -->
 	<!-- tower mount positions | relative to base_link -->
-	<property name="tower_x" value="${def_tower_x+offset_tower_x}"/>
-	<property name="tower_y" value="${def_tower_y+offset_tower_y}"/>
-	<property name="tower_z" value="${def_tower_z+offset_tower_z}"/>
-	<property name="tower_roll" value="${def_tower_roll+offset_tower_roll}"/>
-	<property name="tower_pitch" value="${def_tower_pitch+offset_tower_pitch}"/>
-	<property name="tower_yaw" value="${def_tower_yaw+offset_tower_yaw}"/>
+	<xacro:property name="tower_x" value="${def_tower_x+offset_tower_x}"/>
+	<xacro:property name="tower_y" value="${def_tower_y+offset_tower_y}"/>
+	<xacro:property name="tower_z" value="${def_tower_z+offset_tower_z}"/>
+	<xacro:property name="tower_roll" value="${def_tower_roll+offset_tower_roll}"/>
+	<xacro:property name="tower_pitch" value="${def_tower_pitch+offset_tower_pitch}"/>
+	<xacro:property name="tower_yaw" value="${def_tower_yaw+offset_tower_yaw}"/>
 	<!-- arm mount positions | relative to base_link -->
-	<property name="arm_x" value="${def_arm_x+offset_arm_x}"/>
-	<property name="arm_y" value="${def_arm_y+offset_arm_y}"/>
-	<property name="arm_z" value="${def_arm_z+offset_arm_z}"/>
-	<property name="arm_roll" value="${def_arm_roll+offset_arm_roll}"/>
-	<property name="arm_pitch" value="${def_arm_pitch+offset_arm_pitch}"/>
-	<property name="arm_yaw" value="${def_arm_yaw+offset_arm_yaw}"/>
+	<xacro:property name="arm_x" value="${def_arm_x+offset_arm_x}"/>
+	<xacro:property name="arm_y" value="${def_arm_y+offset_arm_y}"/>
+	<xacro:property name="arm_z" value="${def_arm_z+offset_arm_z}"/>
+	<xacro:property name="arm_roll" value="${def_arm_roll+offset_arm_roll}"/>
+	<xacro:property name="arm_pitch" value="${def_arm_pitch+offset_arm_pitch}"/>
+	<xacro:property name="arm_yaw" value="${def_arm_yaw+offset_arm_yaw}"/>
+	<!-- gripper mount positions | relative to arm_ee_link -->
+    <!--directly defined at ./src/cob_robots/cob_hardware_config/robots/raw3-6/urdf/raw3-6.urdf.xacro-->
+    <!--<xacro:property name="gripper_x" value="${def_gripper_x+offset_gripper_x}"/>-->
+	<!--<xacro:property name="gripper_y" value="${def_gripper_y+offset_gripper_y}"/>-->
+	<!--<xacro:property name="gripper_z" value="${def_gripper_z+offset_gripper_z}"/>-->
+	<!--<xacro:property name="gripper_roll" value="${def_gripper_roll+offset_gripper_roll}"/>-->
+	<!--<xacro:property name="gripper_pitch" value="${def_gripper_pitch+offset_gripper_pitch}"/>-->
+	<!--<xacro:property name="gripper_yaw" value="${def_gripper_yaw+offset_gripper_yaw}"/>-->
 </robot>

File: cob_hardware_config/robots/raw3-6/urdf/raw3-6.urdf.xacro (robot description, xacro)
@@ -1,4 +1,5 @@
 <?xml version="1.0"?>
-<robot xmlns:xacro="http://www.ros.org/wiki/xacro" name="raw3-6" >
+<robot xmlns:xacro="http://www.ros.org/wiki/xacro"
+       name="raw3-6" >
   <!-- common stuff -->
   <xacro:include filename="$(find cob_description)/urdf/common.xacro" />
@@ -10,13 +11,41 @@
   <xacro:include filename="$(find raw_description)/urdf/tower_symetric/tower.urdf.xacro" />
   <!-- ur10 -->
-  <xacro:include filename="$(find raw_description)/urdf/ur_arm/ur10_arm.urdf.xacro" />
+  <xacro:include filename="$(find cob_description)/urdf/ur_arm/ur10_arm.urdf.xacro" />
   <!-- robotiq gripper -->
   <xacro:include filename="$(find robotiq_s_model_visualization)/cfg/robotiq_hand_macro.urdf.xacro" />
   <!-- RealSense Sensors -->
-  <xacro:include filename="$(find cob_description)/urdf/sensors/r200.urdf.xacro"/>
+  <!--<xacro:include filename="$(find cob_description)/urdf/sensors/r200.urdf.xacro"/>-->
   <!-- sick s300 -->
   <xacro:include filename="$(find cob_description)/urdf/sensors/sick_s300_laser.urdf.xacro"/>
   <!-- composition of the robot -->
   <xacro:raw_base name="base"/>
+  <!-- base laser front -->
+  <!--XXX: these parameters are from cob_robots/cob_hardware_config/robots/raw3-5/urdf/properties.urdf.xacro-->
+  <xacro:sick_s300_laser_v0 name="base_laser_front" parent="base">
+    <origin xyz="${laser_front_x} ${laser_front_y} ${laser_front_z}" rpy="${laser_front_roll} ${laser_front_pitch} ${laser_front_yaw}" />
+  </xacro:sick_s300_laser_v0>
+  <!-- base laser rear -->
+  <xacro:sick_s300_laser_v0 name="base_laser_rear" parent="base">
+    <origin xyz="${laser_rear_x} ${laser_rear_y} ${laser_rear_z}" rpy="${laser_rear_roll} ${laser_rear_pitch} ${laser_rear_yaw}" />
+  </xacro:sick_s300_laser_v0>
+  <xacro:tower_symetric name="tower" parent="base_link">
+      <origin xyz="${tower_x} ${tower_y} ${tower_z}" rpy="${tower_roll} ${tower_pitch} ${tower_yaw}" />
+  </xacro:tower_symetric>
+  <xacro:ur10 name="arm" parent="base_link">
+    <origin xyz="${arm_x} ${arm_y} ${arm_z}" rpy="${arm_roll} ${arm_pitch} ${arm_yaw}" />
+  </xacro:ur10>
+  <!--directlt defined here instead of retrieving from-->
+  <!--$(find cob_hardware_config)/robots/raw3-6/urdf/properties.urdf.xacro-->
+  <!--it has to be arm_tool0 instead of arm_ee_link-->
+  <xacro:robotiq_hand prefix="gripper_" parent="arm_tool0" reflect="0">
+    <origin xyz="0 0 .05" rpy="1.570795 0 -0.7753975"/>
+    <!--<origin xyz="0 0 .05" rpy="1.570795 0 -1.570795"/>-->
+  </xacro:robotiq_hand>
+  <!--
+  <xacro:sensor_r200 prefix="vision_wrist_" parent="arm_tool0">
+    <origin xyz="0 -0.3 .15" rpy="1.570795 0 -0.7753975"/>
+  </xacro:sensor_r200>
+  -->
+  <!--
   <gazebo>
     <plugin name="ros_control" filename="libhwi_switch_gazebo_ros_control.so">
@@ -25,27 +54,6 @@
     </plugin>
   </gazebo>
-  <xacro:tower_symetric name="tower" parent="base_link">
-      <origin xyz="${tower_x} ${tower_y} ${tower_z}" rpy="${tower_roll} ${tower_pitch} ${tower_yaw}" />
-  </xacro:tower_symetric>
-  <xacro:ur10 name="arm" parent="base_link">
-    <origin xyz="${arm_x} ${arm_y} ${arm_z}" rpy="${arm_roll} ${arm_pitch} ${arm_yaw}" />
-  </xacro:ur10>
-  <xacro:robotiq_hand prefix="gripper_" parent="arm_tool0" reflect="0">
-    <origin xyz="0 0 .05" rpy="1.570795 0 -0.7753975"/>
-    <!--<origin xyz="0 0 .05" rpy="1.570795 0 -1.570795"/>-->
-  </xacro:robotiq_hand>
-  <!-- sick s300 -->
-  <!--XXX: these parameters are from cob_robots/cob_hardware_config/robots/raw3-5/urdf/properties.urdf.xacro-->
-  <xacro:sick_s300_laser_v0 name="base_laser_front" parent="base">
-    <origin xyz="${laser_front_x} ${laser_front_y} ${laser_front_z}" rpy="${laser_front_roll} ${laser_front_pitch} ${laser_front_yaw}" />
-  </xacro:sick_s300_laser_v0>
-  <xacro:sick_s300_laser_v0 name="base_laser_rear" parent="base">
-    <origin xyz="${laser_rear_x} ${laser_rear_y} ${laser_rear_z}" rpy="${laser_rear_roll} ${laser_rear_pitch} ${laser_rear_yaw}" />
-  </xacro:sick_s300_laser_v0>
+  -->
   <!--
-  <xacro:sensor_r200 prefix="vision_wrist_" parent="arm_tool0">
-    <origin xyz="0 -0.3 .15" rpy="1.570795 0 -0.7753975"/>
-  </xacro:sensor_r200>
-  -->
   <gazebo>
     <plugin name="ros_control" filename="libhwi_switch_gazebo_ros_control.so">
@@ -54,3 +62,4 @@
     </plugin>
   </gazebo>
-  </robot>
+  -->
+</robot>
